Commit message: add new files to be tracked

File: sr_description/hand/xacro/finger/distal/distal.urdf.xacro (robot description, xacro)
@@ -75,4 +75,7 @@
     </xacro:unless>
     <!-- extensions -->
+    <xacro:unless value="${sim_platform == 'gazebo'}">
+      <xacro:distal_transmission />
+    </xacro:unless>
     <xacro:distal_gazebo />
   </xacro:macro>

File: sr_description/hand/xacro/finger/fingers.urdf.xacro (robot description, xacro)
@@ -7,5 +7,5 @@
   <xacro:include filename="$(find sr_description)/hand/xacro/finger/middle/middle_and_distal_bt_2p.urdf.xacro" />
   <xacro:macro name="finger" params="hand_type:=^ hand_version:=^ tip_sensor:=^|pst mid_sensor:=^|none prox_sensor:=^|none reflect:=^ prefix:=^
-                                     link_prefix joint_prefix parent *origin *axis">
+                                     link_prefix joint_prefix parent *origin *axis sim_platform:=^" >
     <!-- Little finger special case -->
     <xacro:if value="${link_prefix == 'lf'}">

File: sr_description/hand/xacro/finger/middle/middle.urdf.xacro (robot description, xacro)
@@ -8,5 +8,6 @@
   <xacro:include filename="$(find sr_description)/hand/xacro/finger/middle/middle.gazebo.xacro" />
   <xacro:include filename="$(find sr_description)/hand/xacro/finger/middle/middle.transmission.xacro" />
-  <xacro:macro name="middle" params="hand_type:=^ hand_version:=^ prefix:=^ link_prefix:=^ joint_prefix:=^ parent">
+  <xacro:include filename="$(find sr_description)/hand/xacro/finger/middle/middle.mujoco.transmission.xacro" />
+  <xacro:macro name="middle" params="hand_type:=^ hand_version:=^ prefix:=^ link_prefix:=^ joint_prefix:=^ parent sim_platform:=^" >
     <link name="${prefix}${link_prefix}middle">
       <inertial>
@@ -55,5 +56,10 @@
     </gazebo>
     <!-- extensions -->
-    <xacro:middle_transmission />
+    <xacro:if value="${sim_platform == 'gazebo'}">
+      <xacro:middle_transmission />
+    </xacro:if>
+    <xacro:unless value="${sim_platform == 'gazebo'}">
+      <xacro:middle_transmission_mujoco />
+    </xacro:unless>
     <xacro:middle_gazebo />
   </xacro:macro>

File: sr_description/hand/xacro/hand.urdf.xacro (robot description, xacro)
@@ -3,5 +3,5 @@
        xmlns:controller="http://playerstage.sourceforge.net/gazebo/xmlschema/#controller"
        xmlns:interface="http://playerstage.sourceforge.net/gazebo/xmlschema/#interface">
-  <xacro:macro name="sr_hand" params="hand_type hand_version side fingers tip_sensors prox_sensors mid_sensors palm_sensor mounting_plate">
+  <xacro:macro name="sr_hand" params="hand_type hand_version side fingers tip_sensors prox_sensors mid_sensors palm_sensor mounting_plate sim_platform">
     <!-- Process hand type, version and side parameters -->
     <xacro:include filename="$(find sr_description)/hand/xacro/process_hand_type_version_side_parameters.xacro" />

File: sr_description/hand/xacro/hand_e.urdf.xacro (robot description, xacro)
@@ -14,5 +14,5 @@
   <!-- palm_sensor: specifies the palm tactile sensor -->
   <xacro:macro name="sr_hand_e" params="hand_version:=^ reflect:=^ prefix:=^ fingers:=^|all tip_sensors:=^|pst
-               prox_sensors:=^|none mid_sensors:=^|none palm_sensor:=^|none mounting_plate:=^|false">
+               prox_sensors:=^|none mid_sensors:=^|none palm_sensor:=^|none mounting_plate:=^|false sim_platform:=^" >
     <!-- Process fingers parameter -->
     <xacro:property name="_all_finger_tokens_" value="${python.set('th ff mf rf lf'.split())}" />
@@ -31,5 +31,5 @@
     <xacro:if value="${'ff' in fingers}">
       <xacro:finger link_prefix="ff" joint_prefix="FF" tip_sensor="${tip_sensors.ff}" prox_sensor="${prox_sensors.ff}"
-                    mid_sensor="${mid_sensors.ff}" parent="${prefix}palm">
+                    mid_sensor="${mid_sensors.ff}" parent="${prefix}palm" >
         <origin xyz="${reflect*0.033} 0 0.095" rpy="0 0 0" />
         <axis xyz="0 ${-1*reflect} 0" />

File: sr_description/mujoco_models/urdfs/sr_hand_e.urdf (robot description, URDF)
Before this commit: robot shadowhand_motor, 33 links, 32 joints
Links:
- link rh_forearm: geometry collision box size=0.07 0.07 0.07; collision mesh filename=package://sr_description/meshes/components/forearm/forearm_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 scale=0.001 0.001 0.001
Joints:
- joint rh_FFJ1: limit lower=0 upper=1.57079632679 effort=4.0 velocity=2.0 -> lower=0 upper=1.5707963267948966 effort=2 velocity=2.0
- joint rh_FFJ2: limit lower=0 upper=1.57079632679 effort=4.0 velocity=2.0 -> lower=0 upper=1.5707963267948966 effort=2 velocity=2.0
- joint rh_FFJ3: limit lower=0 upper=1.57079632679 effort=4.0 velocity=2.0 -> lower=-0.2617993877991494 upper=1.5707963267948966 effort=2 velocity=2.0
- joint rh_FFJ4: axis 0 -1.0 0 -> 0 -1 0; limit lower=-0.349065850399 upper=0.349065850399 effort=4.0 velocity=2.0 -> lower=-0.3490658503988659 upper=0.3490658503988659 effort=2 velocity=2.0
- joint rh_LFJ1: limit lower=0 upper=1.57079632679 effort=4.0 velocity=2.0 -> lower=0 upper=1.5707963267948966 effort=2 velocity=2.0
- joint rh_LFJ2: limit lower=0 upper=1.57079632679 effort=4.0 velocity=2.0 -> lower=0 upper=1.5707963267948966 effort=2 velocity=2.0
- joint rh_LFJ3: limit lower=0 upper=1.57079632679 effort=4.0 velocity=2.0 -> lower=-0.2617993877991494 upper=1.5707963267948966 effort=2 velocity=2.0
- joint rh_LFJ4: axis 0 1.0 0 -> 0 1 0; limit lower=-0.349065850399 upper=0.349065850399 effort=4.0 velocity=2.0 -> lower=-0.3490658503988659 upper=0.3490658503988659 effort=2 velocity=2.0
- joint rh_LFJ5: limit lower=0 upper=0.785398163397 effort=4.0 velocity=2.0 -> lower=0 upper=0.7853981633974483 effort=2 velocity=2.0
- joint rh_MFJ1: limit lower=0 upper=1.57079632679 effort=4.0 velocity=2.0 -> lower=0 upper=1.5707963267948966 effort=2 velocity=2.0
- joint rh_MFJ2: limit lower=0 upper=1.57079632679 effort=4.0 velocity=2.0 -> lower=0 upper=1.5707963267948966 effort=2 velocity=2.0
- joint rh_MFJ3: limit lower=0 upper=1.57079632679 effort=4.0 velocity=2.0 -> lower=-0.2617993877991494 upper=1.5707963267948966 effort=2 velocity=2.0
- joint rh_MFJ4: axis 0 -1.0 0 -> 0 -1 0; limit lower=-0.349065850399 upper=0.349065850399 effort=4.0 velocity=2.0 -> lower=-0.3490658503988659 upper=0.3490658503988659 effort=2 velocity=2.0
- joint rh_RFJ1: limit lower=0 upper=1.57079632679 effort=4.0 velocity=2.0 -> lower=0 upper=1.5707963267948966 effort=2 velocity=2.0
- joint rh_RFJ2: limit lower=0 upper=1.57079632679 effort=4.0 velocity=2.0 -> lower=0 upper=1.5707963267948966 effort=2 velocity=2.0
- joint rh_RFJ3: limit lower=0 upper=1.57079632679 effort=4.0 velocity=2.0 -> lower=-0.2617993877991494 upper=1.5707963267948966 effort=2 velocity=2.0
- joint rh_RFJ4: axis 0 1.0 0 -> 0 1 0; limit lower=-0.349065850399 upper=0.349065850399 effort=4.0 velocity=2.0 -> lower=-0.3490658503988659 upper=0.3490658503988659 effort=2 velocity=2.0
- joint rh_THJ1: limit lower=0 upper=1.57079632679 effort=4.0 velocity=4.0 -> lower=-0.2617993877991494 upper=1.5707963267948966 effort=1.0 velocity=4.0; origin xyz=0 0 0.032 rpy=0 0 -1.57079632679 -> xyz=0 0 0.032 rpy=0 0 -1.5707963267948966
- joint rh_THJ2: limit lower=-0.698131700798 upper=0.698131700798 effort=4.0 velocity=2.0 -> lower=-0.6981317007977318 upper=0.6981317007977318 effort=2.0 velocity=2.0
- joint rh_THJ3: limit lower=-0.209439510239 upper=0.209439510239 effort=4.0 velocity=4.0 -> lower=-0.20943951023931953 upper=0.20943951023931953 effort=2.0 velocity=4.0
- joint rh_THJ4: axis 1.0 0 0 -> 1 0 0; limit lower=0.0 upper=1.2217304764 effort=4.0 velocity=4.0 -> lower=0.0 upper=1.2217304763960306 effort=3 velocity=4.0
- joint rh_THJ5: axis 0 0 -1.0 -> 0 0 -1; limit lower=-1.0471975512 upper=1.0471975512 effort=4.0 velocity=4.0 -> lower=-1.0471975511965976 upper=1.0471975511965976 effort=5.0 velocity=4.0; origin xyz=0.034 -0.0085 0.029 rpy=0 0.785398163397 0.0 -> xyz=0.034 -0.00858 0.029 rpy=0 0.7853981633974483 0.0
- joint rh_WRJ1: limit lower=-0.698131700798 upper=0.488692190558 effort=5.0 velocity=2.0 -> lower=-0.6981317007977318 upper=0.4886921905584123 effort=30 velocity=2.0
- joint rh_WRJ2: axis 0 1.0 0 -> 0 1 0; limit lower=-0.523598775598 upper=0.174532925199 effort=10.0 velocity=2.0 -> lower=-0.5235987755982988 upper=0.17453292519943295 effort=10 velocity=2.0; origin xyz=0 -0.010 0.213 rpy=0 0 0 -> xyz=0 -0.010 0.21301 rpy=0 0 0

File: sr_description/mujoco_models/urdfs/sr_hand_e_test.urdf (robot description, URDF)
Before this commit: robot shadowhand_motor, 33 links, 32 joints
Links:
- link rh_forearm: geometry collision box size=0.07 0.07 0.07; collision cylinder length=0.008 radius=0.0675
Joints:
- joint rh_FFJ1: limit lower=0 upper=1.57079632679 effort=4.0 velocity=2.0 -> lower=0 upper=1.5707963267948966 effort=2 velocity=2.0
- joint rh_FFJ2: limit lower=0 upper=1.57079632679 effort=4.0 velocity=2.0 -> lower=0 upper=1.5707963267948966 effort=2 velocity=2.0
- joint rh_FFJ3: limit lower=0 upper=1.57079632679 effort=4.0 velocity=2.0 -> lower=-0.2617993877991494 upper=1.5707963267948966 effort=2 velocity=2.0
- joint rh_FFJ4: axis 0 -1.0 0 -> 0 -1 0; limit lower=-0.349065850399 upper=0.349065850399 effort=4.0 velocity=2.0 -> lower=-0.3490658503988659 upper=0.3490658503988659 effort=2 velocity=2.0
- joint rh_LFJ1: limit lower=0 upper=1.57079632679 effort=4.0 velocity=2.0 -> lower=0 upper=1.5707963267948966 effort=2 velocity=2.0
- joint rh_LFJ2: limit lower=0 upper=1.57079632679 effort=4.0 velocity=2.0 -> lower=0 upper=1.5707963267948966 effort=2 velocity=2.0
- joint rh_LFJ3: limit lower=0 upper=1.57079632679 effort=4.0 velocity=2.0 -> lower=-0.2617993877991494 upper=1.5707963267948966 effort=2 velocity=2.0
- joint rh_LFJ4: axis 0 1.0 0 -> 0 1 0; limit lower=-0.349065850399 upper=0.349065850399 effort=4.0 velocity=2.0 -> lower=-0.3490658503988659 upper=0.3490658503988659 effort=2 velocity=2.0
- joint rh_LFJ5: limit lower=0 upper=0.785398163397 effort=4.0 velocity=2.0 -> lower=0 upper=0.7853981633974483 effort=2 velocity=2.0
- joint rh_MFJ1: limit lower=0 upper=1.57079632679 effort=4.0 velocity=2.0 -> lower=0 upper=1.5707963267948966 effort=2 velocity=2.0
- joint rh_MFJ2: limit lower=0 upper=1.57079632679 effort=4.0 velocity=2.0 -> lower=0 upper=1.5707963267948966 effort=2 velocity=2.0
- joint rh_MFJ3: limit lower=0 upper=1.57079632679 effort=4.0 velocity=2.0 -> lower=-0.2617993877991494 upper=1.5707963267948966 effort=2 velocity=2.0
- joint rh_MFJ4: axis 0 -1.0 0 -> 0 -1 0; limit lower=-0.349065850399 upper=0.349065850399 effort=4.0 velocity=2.0 -> lower=-0.3490658503988659 upper=0.3490658503988659 effort=2 velocity=2.0
- joint rh_RFJ1: limit lower=0 upper=1.57079632679 effort=4.0 velocity=2.0 -> lower=0 upper=1.5707963267948966 effort=2 velocity=2.0
- joint rh_RFJ2: limit lower=0 upper=1.57079632679 effort=4.0 velocity=2.0 -> lower=0 upper=1.5707963267948966 effort=2 velocity=2.0
- joint rh_RFJ3: limit lower=0 upper=1.57079632679 effort=4.0 velocity=2.0 -> lower=-0.2617993877991494 upper=1.5707963267948966 effort=2 velocity=2.0
- joint rh_RFJ4: axis 0 1.0 0 -> 0 1 0; limit lower=-0.349065850399 upper=0.349065850399 effort=4.0 velocity=2.0 -> lower=-0.3490658503988659 upper=0.3490658503988659 effort=2 velocity=2.0
- joint rh_THJ1: limit lower=0 upper=1.57079632679 effort=4.0 velocity=4.0 -> lower=-0.2617993877991494 upper=1.5707963267948966 effort=1.0 velocity=4.0; origin xyz=0 0 0.032 rpy=0 0 -1.57079632679 -> xyz=0 0 0.032 rpy=0 0 -1.5707963267948966
- joint rh_THJ2: limit lower=-0.698131700798 upper=0.698131700798 effort=4.0 velocity=2.0 -> lower=-0.6981317007977318 upper=0.6981317007977318 effort=2.0 velocity=2.0
- joint rh_THJ3: limit lower=-0.209439510239 upper=0.209439510239 effort=4.0 velocity=4.0 -> lower=-0.20943951023931953 upper=0.20943951023931953 effort=2.0 velocity=4.0
- joint rh_THJ4: axis 1.0 0 0 -> 1 0 0; limit lower=0.0 upper=1.2217304764 effort=4.0 velocity=4.0 -> lower=0.0 upper=1.2217304763960306 effort=3 velocity=4.0
- joint rh_THJ5: axis 0 0 -1.0 -> 0 0 -1; limit lower=-1.0471975512 upper=1.0471975512 effort=4.0 velocity=4.0 -> lower=-1.0471975511965976 upper=1.0471975511965976 effort=5.0 velocity=4.0; origin xyz=0.034 -0.0085 0.029 rpy=0 0.785398163397 0.0 -> xyz=0.034 -0.00858 0.029 rpy=0 0.7853981633974483 0.0
- joint rh_WRJ1: limit lower=-0.698131700798 upper=0.488692190558 effort=5.0 velocity=2.0 -> lower=-0.6981317007977318 upper=0.4886921905584123 effort=30 velocity=2.0
- joint rh_WRJ2: axis 0 1.0 0 -> 0 1 0; limit lower=-0.523598775598 upper=0.174532925199 effort=10.0 velocity=2.0 -> lower=-0.5235987755982988 upper=0.17453292519943295 effort=10 velocity=2.0; origin xyz=0 -0.010 0.213 rpy=0 0 0 -> xyz=0 -0.010 0.21301 rpy=0 0 0
