Commit message: add new files to be tracked

File: sr_description/mujoco_models/urdfs/ur10_hand.urdf (robot description, URDF)
Before this commit: robot ur10srh, 43 links, 42 joints
Links:
- added link ra_base_link_inertia, mass 4.0; collision mesh filename=package://ur_description/meshes/ur10/collision/base.stl; visual mesh filename=package://ur_description/meshes/ur10/visual/base.dae
- link ra_base_link: mass 4.0 -> None; geometry 
- link ra_flange: geometry 
- link rh_ffdistal: geometry collision mesh filename=package://sr_description/meshes/components/f_distal/pst/f_d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 scale=0.001 0.001 0.001; visual mesh filename=package://sr_description/meshes/components/f_distal/pst/f_d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 scale=0.001 0.001 0.001
- link rh_ffknuckle: geometry collision cylinder length=0.014 radius=0.007; visual mesh filename=package://sr_description/meshes/components/f_knuckle/f_knuc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 scale=0.001 0.001 0.001
- link rh_ffmiddle: geometry collision cylinder length=0.025 radius=0.007; collision sphere radius=0.007
- link rh_ffproximal: geometry collision cylinder length=0.040 radius=0.007; visual mesh filename=package://sr_description/meshes/components/f_proximal/f_pro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 scale=0.001 0.001 0.001
- link rh_forearm: geometry collision box size=0.07 0.07 0.07; collision cylinder length=0.008 radius=0.0675
- link rh_lfdistal: geometry collision mesh filename=package://sr_description/meshes/components/f_distal/pst/f_d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 scale=0.001 0.001 0.001; visual mesh filename=package://sr_description/meshes/components/f_distal/pst/f_d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 scale=0.001 0.001 0.001
- link rh_lfknuckle: geometry collision cylinder length=0.014 radius=0.007; visual mesh filename=package://sr_description/meshes/components/f_knuckle/f_knuc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 scale=0.001 0.001 0.001
- link rh_lfmetacarpal: geometry collision box size=0.018 0.024 0.040; visual mesh filename=package://sr_description/meshes/components/lf_metacarpal/lf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 scale=0.001 0.001 0.001
- link rh_lfmiddle: geometry collision cylinder length=0.025 radius=0.007; collision sphere radius=0.007
- link rh_lfproximal: geometry collision cylinder length=0.040 radius=0.007; visual mesh filename=package://sr_description/meshes/components/f_proximal/f_pro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 scale=0.001 0.001 0.001
- link rh_mfdistal: geometry collision mesh filename=package://sr_description/meshes/components/f_distal/pst/f_d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 scale=0.001 0.001 0.001; visual mesh filename=package://sr_description/meshes/components/f_distal/pst/f_d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 scale=0.001 0.001 0.001
- link rh_mfknuckle: geometry collision cylinder length=0.014 radius=0.007; visual mesh filename=package://sr_description/meshes/components/f_knuckle/f_knuc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 scale=0.001 0.001 0.001
- link rh_mfmiddle: geometry collision cylinder length=0.025 radius=0.007; collision sphere radius=0.007
- link rh_mfproximal: geometry collision cylinder length=0.040 radius=0.007; visual mesh filename=package://sr_description/meshes/components/f_proximal/f_pro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 scale=0.001 0.001 0.001
- link rh_palm: geometry collision box size=0.018 0.024 0.004; collision box size=0.020 0.024 0.040
- link rh_rfdistal: geometry collision mesh filename=package://sr_description/meshes/components/f_distal/pst/f_d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 scale=0.001 0.001 0.001; visual mesh filename=package://sr_description/meshes/components/f_distal/pst/f_d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 scale=0.001 0.001 0.001
- link rh_rfknuckle: geometry collision cylinder length=0.014 radius=0.007; visual mesh filename=package://sr_description/meshes/components/f_knuckle/f_knuc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 scale=0.001 0.001 0.001
- link rh_rfmiddle: geometry collision cylinder length=0.025 radius=0.007; collision sphere radius=0.007
- link rh_rfproximal: geometry collision cylinder length=0.040 radius=0.007; visual mesh filename=package://sr_description/meshes/components/f_proximal/f_pro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 scale=0.001 0.001 0.001
- link rh_thdistal: geometry collision mesh filename=package://sr_description/meshes/components/th_distal/pst/th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 scale=0.001 0.001 0.001; visual mesh filename=package://sr_description/meshes/components/th_distal/pst/th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 scale=0.001 0.001 0.001
- link rh_thmiddle: geometry collision cylinder length=0.018 radius=0.011; collision sphere radius=0.011
- link rh_thproximal: geometry collision cylinder length=0.018 radius=0.012; visual mesh filename=package://sr_description/meshes/components/th_proximal/th_p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 scale=0.001 0.001 0.001
- link rh_wrist: geometry collision box size=0.027 0.018 0.010; collision box size=0.027 0.018 0.010
Joints:
- removed joint ra_ee_fixed_joint
- removed joint ra_wrist_3_passive_joint
- added joint ra_base_link-base_link_inertia: type fixed, parent ra_base_link, child ra_base_link_inertia, origin xyz=0 0 0 rpy=0 0 3.141592653589793
- added joint ra_flange-tool0: type fixed, parent ra_flange, child ra_tool0, origin xyz=0 0 0 rpy=1.5707963267948966 0 1.5707963267948966
- added joint ra_wrist_3-flange: type fixed, parent ra_wrist_3_link, child ra_flange, origin xyz=0 0 0 rpy=0 -1.5707963267948966 -1.5707963267948966
- joint ra_arm_to_hand: origin xyz=0.012 0.0 0.0 rpy=1.57079632679 0.0 1.57079632679 -> xyz=0.0 0.0 0.0 rpy=1.5707963267948966 3.141592653589793 1.5707963267948966
- joint ra_base_link-base_fixed_joint: origin xyz=0 0 0 rpy=0 0 -3.14159265359 -> xyz=0 0 0 rpy=0 0 3.141592653589793
- joint ra_elbow_joint: limit lower=-3.14159265359 upper=3.14159265359 effort=150.0 velocity=3.15 -> lower=-3.141592653589793 upper=3.141592653589793 effort=150.0 velocity=3.141592653589793
- joint ra_shoulder_lift_joint: limit lower=-6.28318530718 upper=6.28318530718 effort=330.0 velocity=2.16 -> lower=-6.283185307179586 upper=6.283185307179586 effort=330.0 velocity=2.0943951023931953
- joint ra_shoulder_pan_joint: limit lower=-6.28318530718 upper=6.28318530718 effort=330.0 velocity=2.16 -> lower=-6.283185307179586 upper=6.283185307179586 effort=330.0 velocity=2.0943951023931953; origin xyz=0 0 0.1273 rpy=0 0 3.14159265359 -> xyz=0 0 0.1273 rpy=0 0 0; parent ra_base_link -> ra_base_link_inertia
- joint ra_wrist_1_joint: limit lower=-6.28318530718 upper=6.28318530718 effort=54.0 velocity=3.2 -> lower=-6.283185307179586 upper=6.283185307179586 effort=56.0 velocity=3.141592653589793
- joint ra_wrist_2_joint: limit lower=-6.28318530718 upper=6.28318530718 effort=54.0 velocity=3.2 -> lower=-6.283185307179586 upper=6.283185307179586 effort=56.0 velocity=3.141592653589793; origin xyz=0 -0.1157 -2.37304666792e-11 rpy=1.570796327 0 0 -> xyz=0 -0.1157 -2.373046667922381e-11 rpy=1.570796327 0 0
- joint ra_wrist_3_joint: limit lower=-6.28318530718 upper=6.28318530718 effort=54.0 velocity=3.2 -> lower=-6.283185307179586 upper=6.283185307179586 effort=56.0 velocity=3.141592653589793; origin xyz=0 0.0922 -1.89105361091e-11 rpy=1.57079632659 3.14159265359 3.14159265359 -> xyz=0 0.0922 -1.891053610911353e-11 rpy=1.570796326589793 3.141592653589793 3.141592653589793
- joint rh_FFJ1: limit lower=0 upper=1.57079632679 effort=4 velocity=2.0 -> lower=0 upper=1.5707963267948966 effort=2 velocity=2.0
- joint rh_FFJ2: limit lower=0 upper=1.57079632679 effort=4 velocity=2.0 -> lower=0 upper=1.5707963267948966 effort=2 velocity=2.0
- joint rh_FFJ3: limit lower=-0.261799387799 upper=1.57079632679 effort=4 velocity=2.0 -> lower=-0.2617993877991494 upper=1.5707963267948966 effort=2 velocity=2.0
- joint rh_FFJ4: axis 0 -1.0 0 -> 0 -1 0; limit lower=-0.349065850399 upper=0.349065850399 effort=4 velocity=2.0 -> lower=-0.3490658503988659 upper=0.3490658503988659 effort=2 velocity=2.0
- joint rh_LFJ1: limit lower=0 upper=1.57079632679 effort=4 velocity=2.0 -> lower=0 upper=1.5707963267948966 effort=2 velocity=2.0
- joint rh_LFJ2: limit lower=0 upper=1.57079632679 effort=4 velocity=2.0 -> lower=0 upper=1.5707963267948966 effort=2 velocity=2.0
- joint rh_LFJ3: limit lower=-0.261799387799 upper=1.57079632679 effort=2 velocity=2.0 -> lower=-0.2617993877991494 upper=1.5707963267948966 effort=2 velocity=2.0
- joint rh_LFJ4: axis 0 1.0 0 -> 0 1 0; limit lower=-0.349065850399 upper=0.349065850399 effort=2 velocity=2.0 -> lower=-0.3490658503988659 upper=0.3490658503988659 effort=2 velocity=2.0
- joint rh_LFJ5: limit lower=0 upper=0.785398163397 effort=4 velocity=2.0 -> lower=0 upper=0.7853981633974483 effort=2 velocity=2.0
- joint rh_MFJ1: limit lower=0 upper=1.57079632679 effort=4 velocity=2.0 -> lower=0 upper=1.5707963267948966 effort=2 velocity=2.0
- joint rh_MFJ2: limit lower=0 upper=1.57079632679 effort=4 velocity=2.0 -> lower=0 upper=1.5707963267948966 effort=2 velocity=2.0
- joint rh_MFJ3: limit lower=-0.261799387799 upper=1.57079632679 effort=4 velocity=2.0 -> lower=-0.2617993877991494 upper=1.5707963267948966 effort=2 velocity=2.0
- joint rh_MFJ4: axis 0 -1.0 0 -> 0 -1 0; limit lower=-0.349065850399 upper=0.349065850399 effort=2 velocity=2.0 -> lower=-0.3490658503988659 upper=0.3490658503988659 effort=2 velocity=2.0
- joint rh_RFJ1: limit lower=0 upper=1.57079632679 effort=4 velocity=2.0 -> lower=0 upper=1.5707963267948966 effort=2 velocity=2.0
- joint rh_RFJ2: limit lower=0 upper=1.57079632679 effort=4 velocity=2.0 -> lower=0 upper=1.5707963267948966 effort=2 velocity=2.0
- joint rh_RFJ3: limit lower=-0.261799387799 upper=1.57079632679 effort=2 velocity=2.0 -> lower=-0.2617993877991494 upper=1.5707963267948966 effort=2 velocity=2.0
- joint rh_RFJ4: axis 0 1.0 0 -> 0 1 0; limit lower=-0.349065850399 upper=0.349065850399 effort=2 velocity=2.0 -> lower=-0.3490658503988659 upper=0.3490658503988659 effort=2 velocity=2.0
- joint rh_THJ1: limit lower=-0.261799387799 upper=1.57079632679 effort=1.0 velocity=4.0 -> lower=-0.2617993877991494 upper=1.5707963267948966 effort=1.0 velocity=4.0; origin xyz=0 0 0.032 rpy=0 0 -1.57079632679 -> xyz=0 0 0.032 rpy=0 0 -1.5707963267948966
- joint rh_THJ2: limit lower=-0.698131700798 upper=0.698131700798 effort=2.0 velocity=2.0 -> lower=-0.6981317007977318 upper=0.6981317007977318 effort=2.0 velocity=2.0
- joint rh_THJ3: limit lower=-0.209439510239 upper=0.209439510239 effort=2.0 velocity=4.0 -> lower=-0.20943951023931953 upper=0.20943951023931953 effort=2.0 velocity=4.0
- joint rh_THJ4: axis 1.0 0 0 -> 1 0 0; limit lower=0.0 upper=1.2217304764 effort=3 velocity=4.0 -> lower=0.0 upper=1.2217304763960306 effort=3 velocity=4.0
- joint rh_THJ5: axis 0 0 -1.0 -> 0 0 -1; limit lower=-1.0471975512 upper=1.0471975512 effort=5.0 velocity=4.0 -> lower=-1.0471975511965976 upper=1.0471975511965976 effort=5.0 velocity=4.0; origin xyz=0.034 -0.0085 0.029 rpy=0 0.785398163397 0.0 -> xyz=0.034 -0.00858 0.029 rpy=0 0.7853981633974483 0.0
- joint rh_WRJ1: limit lower=-0.698131700798 upper=0.488692190558 effort=30 velocity=2.0 -> lower=-0.6981317007977318 upper=0.4886921905584123 effort=30 velocity=2.0
- joint rh_WRJ2: axis 0 1.0 0 -> 0 1 0; limit lower=-0.523598775598 upper=0.174532925199 effort=10 velocity=2.0 -> lower=-0.5235987755982988 upper=0.17453292519943295 effort=10 velocity=2.0; origin xyz=0 -0.010 0.213 rpy=0 0 0 -> xyz=0 -0.010 0.21301 rpy=0 0 0
- joint world_joint: origin xyz=0.0 0.0 0.1 rpy=0.0 0.0 0.0 -> xyz=0.0 0.0 0.0 rpy=0.0 0.0 0.0

File: sr_description/mujoco_models/urdfs/ur5_hand.urdf (robot description, URDF)
Before this commit: robot shadowhand_motor, 33 links, 32 joints
Links:
- added link ra_base
- added link ra_base_link
- added link ra_base_link_inertia, mass 4.0; collision mesh filename=package://ur_description/meshes/ur5/collision/base.stl; visual mesh filename=package://ur_description/meshes/ur5/visual/base.dae
- added link ra_flange
- added link ra_forearm_link, mass 2.275; collision mesh filename=package://ur_description/meshes/ur5/collision/forearm.stl; visual mesh filename=package://ur_description/meshes/ur5/visual/forearm.dae
- added link ra_shoulder_link, mass 3.7; collision mesh filename=package://ur_description/meshes/ur5/collision/shoulder.stl; visual mesh filename=package://ur_description/meshes/ur5/visual/shoulder.dae
- added link ra_tool0
- added link ra_upper_arm_link, mass 8.393; collision mesh filename=package://ur_description/meshes/ur5/collision/upperarm.stl; visual mesh filename=package://ur_description/meshes/ur5/visual/upperarm.dae
- added link ra_wrist_1_link, mass 1.219; collision mesh filename=package://ur_description/meshes/ur5/collision/wrist1.stl; visual mesh filename=package://ur_description/meshes/ur5/visual/wrist1.dae
- added link ra_wrist_2_link, mass 1.219; collision mesh filename=package://ur_description/meshes/ur5/collision/wrist2.stl; visual mesh filename=package://ur_description/meshes/ur5/visual/wrist2.dae
- added link ra_wrist_3_link, mass 0.1879; collision mesh filename=package://ur_description/meshes/ur5/collision/wrist3.stl; visual mesh filename=package://ur_description/meshes/ur5/visual/wrist3.dae
- link rh_forearm: geometry collision box size=0.07 0.07 0.07; collision cylinder length=0.008 radius=0.0675
Joints:
- removed joint rh_world_joint
- added joint ra_arm_to_hand: type fixed, parent ra_flange, child rh_forearm, origin xyz=0.0 0.0 0.0 rpy=1.5707963267948966 3.141592653589793 1.5707963267948966
- added joint ra_base_link-base_fixed_joint: type fixed, parent ra_base_link, child ra_base, origin xyz=0 0 0 rpy=0 0 3.141592653589793
- added joint ra_base_link-base_link_inertia: type fixed, parent ra_base_link, child ra_base_link_inertia, origin xyz=0 0 0 rpy=0 0 3.141592653589793
- added joint ra_elbow_joint: type revolute, parent ra_upper_arm_link, child ra_forearm_link, origin xyz=-0.425 0 0 rpy=0 0 0, axis 0 0 1, limit lower=-3.141592653589793 upper=3.141592653589793 effort=150.0 velocity=3.141592653589793
- added joint ra_flange-tool0: type fixed, parent ra_flange, child ra_tool0, origin xyz=0 0 0 rpy=1.5707963267948966 0 1.5707963267948966
- added joint ra_shoulder_lift_joint: type revolute, parent ra_shoulder_link, child ra_upper_arm_link, origin xyz=0 0 0 rpy=1.570796327 0 0, axis 0 0 1, limit lower=-6.283185307179586 upper=6.283185307179586 effort=150.0 velocity=3.141592653589793
- added joint ra_shoulder_pan_joint: type revolute, parent ra_base_link_inertia, child ra_shoulder_link, origin xyz=0 0 0.089159 rpy=0 0 0, axis 0 0 1, limit lower=-6.283185307179586 upper=6.283185307179586 effort=150.0 velocity=3.141592653589793
- added joint ra_wrist_1_joint: type revolute, parent ra_forearm_link, child ra_wrist_1_link, origin xyz=-0.39225 0 0.10915 rpy=0 0 0, axis 0 0 1, limit lower=-6.283185307179586 upper=6.283185307179586 effort=28.0 velocity=3.141592653589793
- added joint ra_wrist_2_joint: type revolute, parent ra_wrist_1_link, child ra_wrist_2_link, origin xyz=0 -0.09465 -1.941303950897609e-11 rpy=1.570796327 0 0, axis 0 0 1, limit lower=-6.283185307179586 upper=6.283185307179586 effort=28.0 velocity=3.141592653589793
- added joint ra_wrist_3-flange: type fixed, parent ra_wrist_3_link, child ra_flange, origin xyz=0 0 0 rpy=0 -1.5707963267948966 -1.5707963267948966
- added joint ra_wrist_3_joint: type revolute, parent ra_wrist_2_link, child ra_wrist_3_link, origin xyz=0 0.0823 -1.688001216681175e-11 rpy=1.570796326589793 3.141592653589793 3.141592653589793, axis 0 0 1, limit lower=-6.283185307179586 upper=6.283185307179586 effort=28.0 velocity=3.141592653589793
- added joint world_joint: type fixed, parent world, child ra_base_link, origin xyz=0.0 0.0 0.0 rpy=0.0 0.0 0.0
- joint rh_FFJ1: limit lower=0 upper=1.57079632679 effort=4.0 velocity=2.0 -> lower=0 upper=1.5707963267948966 effort=2 velocity=2.0
- joint rh_FFJ2: limit lower=0 upper=1.57079632679 effort=4.0 velocity=2.0 -> lower=0 upper=1.5707963267948966 effort=2 velocity=2.0
- joint rh_FFJ3: limit lower=0 upper=1.57079632679 effort=4.0 velocity=2.0 -> lower=-0.2617993877991494 upper=1.5707963267948966 effort=2 velocity=2.0
- joint rh_FFJ4: axis 0 -1.0 0 -> 0 -1 0; limit lower=-0.349065850399 upper=0.349065850399 effort=4.0 velocity=2.0 -> lower=-0.3490658503988659 upper=0.3490658503988659 effort=2 velocity=2.0
- joint rh_LFJ1: limit lower=0 upper=1.57079632679 effort=4.0 velocity=2.0 -> lower=0 upper=1.5707963267948966 effort=2 velocity=2.0
- joint rh_LFJ2: limit lower=0 upper=1.57079632679 effort=4.0 velocity=2.0 -> lower=0 upper=1.5707963267948966 effort=2 velocity=2.0
- joint rh_LFJ3: limit lower=0 upper=1.57079632679 effort=4.0 velocity=2.0 -> lower=-0.2617993877991494 upper=1.5707963267948966 effort=2 velocity=2.0
- joint rh_LFJ4: axis 0 1.0 0 -> 0 1 0; limit lower=-0.349065850399 upper=0.349065850399 effort=4.0 velocity=2.0 -> lower=-0.3490658503988659 upper=0.3490658503988659 effort=2 velocity=2.0
- joint rh_LFJ5: limit lower=0 upper=0.785398163397 effort=4.0 velocity=2.0 -> lower=0 upper=0.7853981633974483 effort=2 velocity=2.0
- joint rh_MFJ1: limit lower=0 upper=1.57079632679 effort=4.0 velocity=2.0 -> lower=0 upper=1.5707963267948966 effort=2 velocity=2.0
- joint rh_MFJ2: limit lower=0 upper=1.57079632679 effort=4.0 velocity=2.0 -> lower=0 upper=1.5707963267948966 effort=2 velocity=2.0
- joint rh_MFJ3: limit lower=0 upper=1.57079632679 effort=4.0 velocity=2.0 -> lower=-0.2617993877991494 upper=1.5707963267948966 effort=2 velocity=2.0
- joint rh_MFJ4: axis 0 -1.0 0 -> 0 -1 0; limit lower=-0.349065850399 upper=0.349065850399 effort=4.0 velocity=2.0 -> lower=-0.3490658503988659 upper=0.3490658503988659 effort=2 velocity=2.0
- joint rh_RFJ1: limit lower=0 upper=1.57079632679 effort=4.0 velocity=2.0 -> lower=0 upper=1.5707963267948966 effort=2 velocity=2.0
- joint rh_RFJ2: limit lower=0 upper=1.57079632679 effort=4.0 velocity=2.0 -> lower=0 upper=1.5707963267948966 effort=2 velocity=2.0
- joint rh_RFJ3: limit lower=0 upper=1.57079632679 effort=4.0 velocity=2.0 -> lower=-0.2617993877991494 upper=1.5707963267948966 effort=2 velocity=2.0
- joint rh_RFJ4: axis 0 1.0 0 -> 0 1 0; limit lower=-0.349065850399 upper=0.349065850399 effort=4.0 velocity=2.0 -> lower=-0.3490658503988659 upper=0.3490658503988659 effort=2 velocity=2.0
- joint rh_THJ1: limit lower=0 upper=1.57079632679 effort=4.0 velocity=4.0 -> lower=-0.2617993877991494 upper=1.5707963267948966 effort=1.0 velocity=4.0; origin xyz=0 0 0.032 rpy=0 0 -1.57079632679 -> xyz=0 0 0.032 rpy=0 0 -1.5707963267948966
- joint rh_THJ2: limit lower=-0.698131700798 upper=0.698131700798 effort=4.0 velocity=2.0 -> lower=-0.6981317007977318 upper=0.6981317007977318 effort=2.0 velocity=2.0
- joint rh_THJ3: limit lower=-0.209439510239 upper=0.209439510239 effort=4.0 velocity=4.0 -> lower=-0.20943951023931953 upper=0.20943951023931953 effort=2.0 velocity=4.0
- joint rh_THJ4: axis 1.0 0 0 -> 1 0 0; limit lower=0.0 upper=1.2217304764 effort=4.0 velocity=4.0 -> lower=0.0 upper=1.2217304763960306 effort=3 velocity=4.0
- joint rh_THJ5: axis 0 0 -1.0 -> 0 0 -1; limit lower=-1.0471975512 upper=1.0471975512 effort=4.0 velocity=4.0 -> lower=-1.0471975511965976 upper=1.0471975511965976 effort=5.0 velocity=4.0; origin xyz=0.034 -0.0085 0.029 rpy=0 0.785398163397 0.0 -> xyz=0.034 -0.00858 0.029 rpy=0 0.7853981633974483 0.0
- joint rh_WRJ1: limit lower=-0.698131700798 upper=0.488692190558 effort=5.0 velocity=2.0 -> lower=-0.6981317007977318 upper=0.4886921905584123 effort=30 velocity=2.0
- joint rh_WRJ2: axis 0 1.0 0 -> 0 1 0; limit lower=-0.523598775598 upper=0.174532925199 effort=10.0 velocity=2.0 -> lower=-0.5235987755982988 upper=0.17453292519943295 effort=10 velocity=2.0; origin xyz=0 -0.010 0.213 rpy=0 0 0 -> xyz=0 -0.010 0.21301 rpy=0 0 0

File: sr_description/robots/sr_hand.urdf.xacro (robot description, xacro)
@@ -16,5 +16,6 @@
   <xacro:arg name="palm_sensor" default="none"/>
   <xacro:arg name="mounting_plate" default="false"/>
-  <link name="world" />
+  <xacro:arg name="sim_platform" default="gazebo"/>
+  <link name="world"/>
   <xacro:if value="${'$(arg side)' == 'right'}">
     <joint name="rh_world_joint" type="fixed">
@@ -33,4 +34,4 @@
   <xacro:sr_hand hand_type="$(arg hand_type)" hand_version="$(arg hand_version)" side="$(arg side)"
                  fingers="$(arg fingers)" tip_sensors="$(arg tip_sensors)" mid_sensors="$(arg mid_sensors)"
-                 prox_sensors="$(arg prox_sensors)" palm_sensor="$(arg palm_sensor)" mounting_plate="$(arg mounting_plate)"/>
+                 prox_sensors="$(arg prox_sensors)" palm_sensor="$(arg palm_sensor)" mounting_plate="$(arg mounting_plate)" sim_platform="$(arg sim_platform)"/>
 </robot>
